Commit message: add features

File: rasbot_description/urdf/p3dx_base.urdf.xacro (robot description, xacro)
@@ -5,11 +5,5 @@
   <xacro:macro name="p3dx_base" params="name">
     <link name="base_link">
-      <inertial>
-        <mass value="3.5"/>
-        <origin xyz="0 0 0"/>
-        <inertia ixx="1" ixy="0" ixz="0"
-                 iyy="1" iyz="0"
-                 izz="1"/>
-      </inertial>
+      <xacro:box_inertial x="0.36" y="0.26" z="0.18" mass="9.0" />
       <visual>
         <origin xyz="-0.045 0 0.148" rpy="0 0 0"/>
@@ -20,18 +14,12 @@
       </visual>
       <collision>
-        <origin xyz="0 0 0"/>
+        <origin xyz="-0.045 0 0.148" rpy="0 0 0"/>
         <geometry>
-          <box size="0.01 0.01 0.01"/>
+          <mesh filename="package://rasbot_description/meshes/p3dx/chassis.stl"/>
         </geometry>
       </collision>
     </link>
      <link name="top_plate">
-      <inertial>
-        <mass value="0.01"/>
-        <origin xyz="0 0 0"/>
-        <inertia ixx="1" ixy="0" ixz="0"
-                 iyy="1" iyz="0"
-                 izz="1"/>
-      </inertial>
+      <xacro:box_inertial x="0.445" y="0.38" z="0.01" mass="1.0" />
       <visual>
         <origin xyz="0 0 0"/>
@@ -41,4 +29,10 @@
         <material name="TopBlack"/>
       </visual>
+      <collision>
+        <origin xyz="0.0 0 0.0" rpy="0 0 0"/>
+        <geometry>
+          <mesh filename="package://rasbot_description/meshes/p3dx/top.stl"/>
+        </geometry>
+      </collision>
     </link>
     <joint name="base_top_joint" type="fixed">

File: rasbot_description/urdf/p3dx_caster.urdf.xacro (robot description, xacro)
@@ -21,5 +21,5 @@
         <origin xyz="0 0 0"/>
         <geometry>
-          <cylinder radius="0.03" length="0.02"/>
+          <box size="0.01 0.01 0.01"/>
         </geometry>
       </collision>
@@ -30,4 +30,6 @@
       <child link="caster_swivel"/>
       <axis xyz="0 0 1"/>
+      <dynamics damping="0.0" friction="0.0"/>
+      <limit effort="100" velocity="100" k_velocity="0"/>
     </joint>
     <!-- Center wheel -->
@@ -59,4 +61,6 @@
       <child link="caster_wheel"/>
       <axis xyz="0 1 0"/>
+      <limit effort="100" velocity="100" k_velocity="0"/>
+      <dynamics damping="0.0" friction="0.0"/>
     </joint>
     <!-- Center hubcap -->
@@ -79,5 +83,5 @@
         <origin xyz="0 0 0"/>
         <geometry>
-          <box size="0.05 0.05 0.05"/>
+          <box size="0.01 0.01 0.01"/>
         </geometry>
       </collision>

File: rasbot_description/urdf/p3dx_materials.urdf.xacro (robot description, xacro)
@@ -21,3 +21,24 @@
     </material>
   </xacro:macro>
+  <xacro:macro name="sphere_inertial" params="radius mass">
+    <inertial>
+      <mass value="${mass}" />
+      <origin xyz="0 0 0" />
+      <inertia ixx="${0.4 * mass * radius * radius}" ixy="0.0" ixz="0.0" iyy="${0.4 * mass * radius * radius}" iyz="0.0" izz="${0.4 * mass * radius * radius}" />
+    </inertial>
+  </xacro:macro>
+  <xacro:macro name="cylinder_inertial" params="radius length mass">
+    <inertial>
+      <mass value="${mass}" />
+      <origin xyz="0 0 0" />
+      <inertia ixx="${0.0833333 * mass * (3 * radius * radius + length * length)}" ixy="0.0" ixz="0.0" iyy="${0.0833333 * mass * (3 * radius * radius + length * length)}" iyz="0.0" izz="${0.5 * mass * radius * radius}" />
+    </inertial>
+  </xacro:macro>
+  <xacro:macro name="box_inertial" params="x y z mass">
+    <inertial>
+      <mass value="${mass}" />
+      <origin xyz="0 0 0" />
+      <inertia ixx="${0.0833333 * mass * (y*y + z*z)}" ixy="0.0" ixz="0.0" iyy="${0.0833333 * mass * (x*x + z*z)}" iyz="0.0" izz="${0.0833333 * mass * (x*x + y*y)}" />
+    </inertial>
+  </xacro:macro>
 </robot>

File: rasbot_description/urdf/p3dx_sonars.urdf.xacro (robot description, xacro)
@@ -53,5 +53,5 @@
         <origin xyz="0 0 0"/>
         <geometry>
-          <box size="0.5 0.25 0.05"/>
+           <box size="0.01 0.01 0.01"/>
         </geometry>
       </collision>

File: rasbot_description/urdf/p3dx_wheels.urdf.xacro (robot description, xacro)
@@ -21,5 +21,5 @@
       <origin xyz="0 0 0" rpy="${-3.14159/2} 0 0"/>
       <geometry>
-        <cylinder radius="0.09" length="0.02"/>
+        <cylinder radius="0.09" length="0.01"/>
       </geometry>
     </collision>
@@ -60,4 +60,5 @@
     <child link="p3dx_${suffix}_wheel"/>
     <axis xyz="0 1 0"/>
+    <dynamics damping="0.01" friction="0.0"/>
   </joint>
 </xacro:macro>
