Commit message: [FEAT] Add LIDAR

File: p3dx_gazebo/urdf/p3dx_gz.urdf.xacro (robot description, xacro)
@@ -27,4 +27,33 @@
         </plugin>
     </gazebo>
+    <gazebo reference="rplidar_link">
+      <sensor name="sensor_ray_front" type="gpu_lidar">
+        <gz_frame_id>rplidar_link</gz_frame_id>
+        <always_on>true</always_on>
+        <visualize>true</visualize>
+        <update_rate>5.0</update_rate>
+        <topic>scan</topic>
+        <lidar>
+          <scan>
+            <horizontal>
+              <samples>360</samples>
+              <resolution>1.000000</resolution>
+              <min_angle>0.000000</min_angle>
+              <max_angle>6.280000</max_angle>
+            </horizontal>
+          </scan>
+          <range>
+            <min>0.120000</min>
+            <max>3.5</max>
+            <resolution>0.015000</resolution>
+          </range>
+          <noise>
+            <type>gaussian</type>
+            <mean>0.0</mean>
+            <stddev>0.01</stddev>
+          </noise>
+        </lidar>
+      </sensor>
+    </gazebo>
     <xacro:include filename="$(find p3dx_gazebo)/urdf/robot_material_support.xacro"/>
 </robot>

File: rasbot_description/urdf/p3dx.urdf.xacro (robot description, xacro)
@@ -6,8 +6,17 @@
   <xacro:include filename="$(find rasbot_description)/urdf/p3dx_caster.urdf.xacro"/>
   <xacro:include filename="$(find rasbot_description)/urdf/p3dx_sonars.urdf.xacro"/>
+  <xacro:include filename="$(find rasbot_description)/urdf/rplidar_macro.urdf.xacro"/>
   <xacro:p3dx_base name="p3dx"/>
-  <xacro:p3dx_wheel suffix="left"  reflect="-1"/>
-  <xacro:p3dx_wheel suffix="right" reflect="1"/>
+  <xacro:p3dx_wheel suffix="left"  reflect="1"/>
+  <xacro:p3dx_wheel suffix="right" reflect="-1"/>
   <xacro:p3dx_caster/>
   <xacro:p3dx_sonars/>
+  <xacro:rplidar
+        name="rplidar"
+        parent_link="top_plate"
+        mass="0.01"
+        radius="0.015"
+        length="0.01">
+    <origin xyz="0.15 0.0 0.047" rpy="0 0 ${pi}"/>
+  </xacro:rplidar>
 </robot>

Commit message: [FEAT] add navsat

File: p3dx_gazebo/urdf/p3dx_gz.urdf.xacro (robot description, xacro)
@@ -1,69 +1,145 @@
 <?xml version="1.0"?>
 <robot xmlns:xacro="http://www.ros.org/wiki/xacro" name="p3dx">
-    <xacro:include filename="$(find rasbot_description)/urdf/p3dx.urdf.xacro"/>
-    <gazebo>
-        <plugin filename="gz-sim-diff-drive-system"
-                name="gz::sim::systems::DiffDrive">
-            <left_joint>p3dx_left_wheel_joint</left_joint>
-            <right_joint>p3dx_right_wheel_joint</right_joint>
-            <wheel_separation>0.31</wheel_separation>
-            <wheel_radius>0.0868</wheel_radius>
-            <topic>cmd_vel</topic>
-            <odom_topic>/unused/diff_drive_odometry</odom_topic>
-             <tf_topic>/unused/diff_drive_tf</tf_topic>
-            <frame_id>odom_diff_drive</frame_id>
-            <child_frame_id>base_link</child_frame_id>
-            <odom_publish_frequency>1</odom_publish_frequency>
-        </plugin>
-    </gazebo>
-    <gazebo>
-      <plugin
-        filename="gz-sim-odometry-publisher-system"
-        name="gz::sim::systems::OdometryPublisher">
-        <odom_publish_frequency>20</odom_publish_frequency>
-        <robot_base_frame>base_link</robot_base_frame>
-        <odom_frame>odom</odom_frame>
-        <odom_topic>odom</odom_topic>
+  <xacro:include filename="$(find rasbot_description)/urdf/p3dx.urdf.xacro"/>
+  <gazebo>
+      <plugin filename="gz-sim-diff-drive-system"
+              name="gz::sim::systems::DiffDrive">
+          <left_joint>p3dx_left_wheel_joint</left_joint>
+          <right_joint>p3dx_right_wheel_joint</right_joint>
+          <wheel_separation>0.31</wheel_separation>
+          <wheel_radius>0.0868</wheel_radius>
+          <topic>cmd_vel</topic>
+          <odom_topic>/unused/diff_drive_odometry</odom_topic>
+            <tf_topic>/unused/diff_drive_tf</tf_topic>
+          <frame_id>odom_diff_drive</frame_id>
+          <child_frame_id>base_link</child_frame_id>
+          <odom_publish_frequency>1</odom_publish_frequency>
       </plugin>
-    </gazebo>
-    <gazebo>
-        <plugin filename="gz-sim-joint-state-publisher-system"
-                name="gz::sim::systems::JointStatePublisher">
-            <topic>joint_states</topic>
-            <joint_name>p3dx_left_wheel_joint</joint_name>
-            <joint_name>p3dx_right_wheel_joint</joint_name>
-            <joint_name>base_caster_swivel_joint</joint_name>
-            <joint_name>caster_swivel_wheel_joint</joint_name>
-        </plugin>
-    </gazebo>
-    <gazebo reference="rplidar_link">
-      <sensor name="sensor_ray_front" type="gpu_lidar">
-        <gz_frame_id>rplidar_link</gz_frame_id>
+  </gazebo>
+  <gazebo>
+    <plugin
+      filename="gz-sim-odometry-publisher-system"
+      name="gz::sim::systems::OdometryPublisher">
+      <odom_publish_frequency>20</odom_publish_frequency>
+      <robot_base_frame>base_link</robot_base_frame>
+      <odom_frame>odom</odom_frame>
+      <odom_topic>odom</odom_topic>
+    </plugin>
+  </gazebo>
+  <gazebo>
+      <plugin filename="gz-sim-joint-state-publisher-system"
+              name="gz::sim::systems::JointStatePublisher">
+          <topic>joint_states</topic>
+          <joint_name>p3dx_left_wheel_joint</joint_name>
+          <joint_name>p3dx_right_wheel_joint</joint_name>
+          <joint_name>base_caster_swivel_joint</joint_name>
+          <joint_name>caster_swivel_wheel_joint</joint_name>
+      </plugin>
+  </gazebo>
+  <gazebo reference="rplidar_link">
+    <sensor name="sensor_ray_front" type="gpu_lidar">
+      <gz_frame_id>rplidar_link</gz_frame_id>
+      <always_on>true</always_on>
+      <visualize>true</visualize>
+      <update_rate>10.0</update_rate>
+      <topic>scan</topic>
+      <lidar>
+        <scan>
+          <horizontal>
+            <samples>720</samples>
+            <resolution>1</resolution>
+            <min_angle>-3.14159265</min_angle>
+            <max_angle>3.14159265</max_angle>
+          </horizontal>
+        </scan>
+        <range>
+          <min>0.20</min>
+          <max>12.0</max>
+          <resolution>0.01</resolution>
+        </range>
+        <noise>
+          <type>gaussian</type>
+          <mean>0.0</mean>
+          <stddev>0.01</stddev>
+        </noise>
+      </lidar>
+    </sensor>
+  </gazebo>
+  <gazebo reference="gps_link">
+    <sensor name="navsat" type="navsat">
+      <always_on>true</always_on>
+      <update_rate>1</update_rate>
+      <topic>gps/fix</topic>
+      <gz_frame_id>gps_link</gz_frame_id>
+      <navsat>
+        <position_sensing>
+          <horizontal>
+          <!-- Be carefull setting this.
+          Units in degree not in meters https://github.com/gazebosim/sdformat/issues/1572 -->
+            <noise type="gaussian">
+              <mean>0.0</mean>
+              <stddev>0.0</stddev>
+            </noise>
+          </horizontal>
+          <vertical>
+            <noise type="gaussian">
+              <mean>0.0</mean>
+              <stddev>0.0</stddev>
+            </noise>
+          </vertical>
+        </position_sensing>
+      </navsat>
+    </sensor>
+  </gazebo>
+  <gazebo reference="imu_link">
+    <sensor name="p3dx_imu" type="imu">
         <always_on>true</always_on>
-        <visualize>true</visualize>
-        <update_rate>10.0</update_rate>
-        <topic>scan</topic>
-        <lidar>
-          <scan>
-            <horizontal>
-              <samples>720</samples>
-              <resolution>1</resolution>
-              <min_angle>-3.14159265</min_angle>
-              <max_angle>3.14159265</max_angle>
-            </horizontal>
-          </scan>
-          <range>
-            <min>0.20</min>
-            <max>12.0</max>
-            <resolution>0.01</resolution>
-          </range>
-          <noise>
-            <type>gaussian</type>
-            <mean>0.0</mean>
-            <stddev>0.01</stddev>
-          </noise>
-        </lidar>
+        <update_rate>200</update_rate>
+        <topic>imu/data</topic>
+        <gz_frame_id>imu_link</gz_frame_id>
+        <imu>
+          <angular_velocity>
+            <x>
+              <noise type="gaussian">
+                <mean>0.0</mean>
+                <stddev>2e-4</stddev>
+              </noise>
+            </x>
+            <y>
+              <noise type="gaussian">
+                <mean>0.0</mean>
+                <stddev>2e-4</stddev>
+              </noise>
+            </y>
+            <z>
+              <noise type="gaussian">
+                <mean>0.0</mean>
+                <stddev>2e-4</stddev>
+              </noise>
+            </z>
+          </angular_velocity>
+          <linear_acceleration>
+            <x>
+              <noise type="gaussian">
+                <mean>0.0</mean>
+                <stddev>1.7e-2</stddev>
+              </noise>
+            </x>
+            <y>
+              <noise type="gaussian">
+                <mean>0.0</mean>
+                <stddev>1.7e-2</stddev>
+              </noise>
+            </y>
+            <z>
+              <noise type="gaussian">
+                <mean>0.0</mean>
+                <stddev>1.7e-2</stddev>
+              </noise>
+            </z>
+          </linear_acceleration>
+        </imu>
       </sensor>
-    </gazebo>
-    <xacro:include filename="$(find p3dx_gazebo)/urdf/robot_material_support.xacro"/>
+  </gazebo>
+  <xacro:include filename="$(find p3dx_gazebo)/urdf/robot_material_support.xacro"/>
 </robot>

File: rasbot_description/urdf/p3dx.urdf.xacro (robot description, xacro)
@@ -20,3 +20,15 @@
     <origin xyz="0.15 0.0 0.047" rpy="0 0 ${pi}"/>
   </xacro:rplidar>
+   <link name="gps_link"/>
+  <joint name="gps_joint" type="fixed">
+      <origin xyz="-0.05 0 0.05" rpy="0 0 0"/>
+      <parent link="base_link"/>
+      <child link="gps_link"/>
+  </joint>
+  <link name="imu_link"/>
+  <joint name="imu_joint" type="fixed">
+      <parent link="base_link"/>
+      <child link="imu_link"/>
+      <origin xyz="0.0 0 0.068" rpy="0 0 0"/>
+  </joint>
 </robot>
